Commit message: Initial Commit

File: nanovoxmap_example/urdf/depth_camera.xacro (robot description, xacro)
@@ -4,5 +4,5 @@
         <origin xyz="0.18 0 0" rpy="0 0 0" />
         <parent link="mid_mount" />
-        <child link="realsense_bracket_link" />
+        <child  link="realsense_bracket_link" />
     </joint>
     <link name="realsense_bracket_link">
@@ -10,79 +10,86 @@
             <origin xyz="0.010 -0.0325 0" rpy="0 0 ${pi/2}" />
             <geometry>
-                <mesh filename="file://$(find nanovoxmap_example)/meshes/mounting_bracket.stl" scale="0.001 0.001 0.001"/>
+                <mesh filename="package://nanovoxmap_example/meshes/mounting_bracket.stl" scale="0.001 0.001 0.001"/>
             </geometry>
-            <material name="aluminum" />
+            <material name="dark_grey" />
         </visual>
+        <collision>
+            <origin xyz="0 0 0.0145" rpy="0 0 0" />
+            <geometry><box size="0.020 0.065 0.029"/></geometry>
+        </collision>
+        <inertial>
+            <mass value="1e-6" />
+            <origin xyz="0 0 0" rpy="0 0 0"/>
+            <inertia ixx="1e-6" ixy="0" ixz="0" iyy="1e-6" iyz="0" izz="1e-6" />
+        </inertial>
     </link>
-    <!-- realsense camera joints -->
+    <!-- Camera body at the plate hole-centre, facing robot +X -->
     <joint type="fixed" name="front_realsense_chassis_joint">
         <origin xyz="-0.007 0 0.022" rpy="0 0 0" />
         <parent link="realsense_bracket_link" />
-        <child link="front_realsense_chassis" />
+        <child  link="front_realsense_chassis" />
     </joint>
     <link name="front_realsense_chassis">
         <visual>
-            <origin xyz="0.025 0 0" rpy="${pi/2} 0 ${pi/2}" />
+            <origin xyz="0.025 0 0" rpy="${-pi/2} 0 ${-pi/2}" />
             <geometry>
-                <mesh filename="file://$(find nanovoxmap_example)/meshes/d435.dae"/>
+                <mesh filename="package://nanovoxmap_example/meshes/d435.dae"/>
             </geometry>
         </visual>
     </link>
-    <joint type="fixed" name="front_realsense_optical_joint">
-        <origin xyz="0.025 0.0 0.0" rpy="0 0 0" />
+    <!-- optical body frame (front glass); Gazebo sensor lives here -->
+    <joint type="fixed" name="front_realsense_joint">
+        <origin xyz="0.025 0 0" rpy="0 0 0" />
         <parent link="front_realsense_chassis" />
-        <child link="front_realsense_optical_link" />
+        <child  link="front_realsense_lens" />
+    </joint>
+    <link name="front_realsense_lens" />
+    <!-- optical frame, REP-103 (z forward, x right, y down) -->
+    <joint name="front_realsense_optical_link_joint" type="fixed">
+        <parent link="front_realsense_lens" />
+        <child  link="front_realsense_optical_link" />
+        <origin xyz="0 0 0" rpy="${-pi/2} 0 ${-pi/2}" />
     </joint>
     <link name="front_realsense_optical_link" />
-    <gazebo reference="front_realsense_optical_link">
-        <sensor name="front_realsense_depth" type="rgbd_camera">
-            <pose>0 0 0 0 0 0</pose>
+    <!-- Gazebo materials (drop the chassis one if the .dae carries its own colours) -->
+    <gazebo reference="realsense_bracket_link"><material>Gazebo/DarkGrey</material></gazebo>
+    <!-- Depth camera -->
+    <gazebo reference="front_realsense_lens">
+        <sensor type="depth" name="front_realsense_depth">
+            <always_on>true</always_on>
+            <update_rate>30</update_rate>
             <camera>
                 <horizontal_fov>1.5184351666666667</horizontal_fov>
-                <vertical_fov>1.0122901111111111</vertical_fov>
                 <image>
                     <width>640</width>
                     <height>480</height>
-                    <format>RGB_INT8</format>
+                    <format>R8G8B8</format>
                 </image>
-                <clip>
-                    <near>0.1</near>
-                    <far>5</far>
-                </clip>
-                <distortion>
-                    <k1>0.0</k1>
-                    <k2>0.0</k2>
-                    <k3>0.0</k3>
-                    <p1>0.0</p1>
-                    <p2>0.0</p2>
-                    <center>0.5 0.5</center>
-                </distortion>
-                <lens>
-                    <intrinsics>
-                        <fx>554.25469</fx>
-                        <fy>554.25469</fy>
-                        <cx>320.5</cx>
-                        <cy>240.5</cy>
-                        <s>0</s>
-                    </intrinsics>
-                </lens>
-                <noise>
-                    <type>gaussian</type>
-                    <mean>0</mean>
-                    <stddev>0.007</stddev>
-                </noise>
-                <depth_camera>
-                    <clip>
-                        <near>0.1</near>
-                        <far>5</far>
-                    </clip>
-                </depth_camera>
+                <clip><near>0.1</near><far>50.0</far></clip>
             </camera>
-            <always_on>1</always_on>
-            <update_rate>30</update_rate>
-            <visualize>true</visualize>
-            <topic>jackal/realsense</topic>
-            <enable_metrics>true</enable_metrics>
-            <gz_frame_id>front_realsense_optical_link</gz_frame_id>
+            <plugin name="realsense_controller" filename="libgazebo_ros_openni_kinect.so">
+                <baseline>0.05</baseline>
+                <alwaysOn>true</alwaysOn>
+                <updateRate>30</updateRate>
+                <cameraName>jackal/realsense</cameraName>
+                <imageTopicName>color/image_raw</imageTopicName>
+                <cameraInfoTopicName>color/camera_info</cameraInfoTopicName>
+                <depthImageTopicName>depth/image_rect_raw</depthImageTopicName>
+                <depthImageInfoTopicName>depth/camera_info</depthImageInfoTopicName>
+                <pointCloudTopicName>depth/color/points</pointCloudTopicName>
+                <frameName>front_realsense_optical_link</frameName>
+                <pointCloudCutoff>0.105</pointCloudCutoff>
+                <pointCloudCutoffMax>8.0</pointCloudCutoffMax>
+                <distortionK1>0</distortionK1>
+                <distortionK2>0</distortionK2>
+                <distortionK3>0</distortionK3>
+                <distortionT1>0</distortionT1>
+                <distortionT2>0</distortionT2>
+                <CxPrime>0</CxPrime>
+                <Cx>0</Cx>
+                <Cy>0</Cy>
+                <focalLength>0</focalLength>
+                <hackBaseline>0</hackBaseline>
+            </plugin>
         </sensor>
     </gazebo>

File: nanovoxmap_example/urdf/jackal.urdf.xacro (robot description, xacro)
@@ -10,10 +10,9 @@
   <xacro:property name="chassis_width" value="0.310" />
   <xacro:property name="chassis_height" value="0.184" />
-  <xacro:include filename="$(find nanovoxmap_example)/urdf/wheel.xacro" />
   <material name="dark_grey">
     <color rgba="0.2 0.2 0.2 1.0"/>
   </material>
-  <material name="aluminum">
-    <color rgba="0.66 0.67 0.71 1.0"/>
+  <material name="light_grey">
+    <color rgba="0.4 0.4 0.4 1.0"/>
   </material>
   <material name="yellow">
@@ -34,5 +33,5 @@
       <origin xyz="0 0 ${footprint_vertical_offset}" rpy="${pi/2} 0 ${pi/2}"/>
       <geometry>
-        <mesh filename="file://$(find nanovoxmap_example)/meshes/jackal-base.stl"/>
+        <mesh filename="package://nanovoxmap_example/meshes/jackal-base.stl"/>
       </geometry>
       <material name="dark_grey" />
@@ -45,9 +44,56 @@
     </collision>
     <inertial>
+      <!-- Center of mass -->
       <origin xyz="0.012  0.002 0.067" rpy="0 0 0"/>
       <mass value="16.523"/>
+      <!-- Moments of inertia: ( chassis without wheels ) -->
       <inertia ixx="0.3136" ixy="-0.0008" ixz="0.0164" iyy="0.3922" iyz="-0.0009" izz="0.4485"/>
     </inertial>
   </link>
+  <gazebo reference="chassis_link">
+    <material>Gazebo/DarkGrey</material>
+  </gazebo>
+  <xacro:macro name="wheel" params="prefix *joint_pose">
+    <link name="${prefix}_wheel_link">
+      <visual>
+        <origin xyz="0 0 0" rpy="${pi/2} 0 0"/>
+        <geometry>
+          <mesh filename="package://nanovoxmap_example/meshes/jackal-wheel.stl"/>
+        </geometry>
+        <material name="black" />
+      </visual>
+      <collision>
+        <origin xyz="0 0 0" rpy="${pi/2} 0 0"/>
+        <geometry>
+          <cylinder radius="${wheel_radius}" length="${wheel_width}"/>
+        </geometry>
+      </collision>
+      <inertial>
+        <origin xyz="0 0 0" rpy="0 0 0"/>
+        <mass value="0.477"/>
+        <inertia ixx="0.0013" ixy="0" ixz="0" iyy="0.0024" iyz="0" izz="0.0013"/>
+      </inertial>
+    </link>
+    <gazebo reference="${prefix}_wheel_link">
+      <material>Gazebo/DarkGrey</material>
+    </gazebo>
+    <joint name="${prefix}_wheel" type="continuous">
+      <parent link="chassis_link"/>
+      <child link="${prefix}_wheel_link" />
+      <xacro:insert_block name="joint_pose" />
+      <axis xyz="0 1 0" />
+    </joint>
+    <!-- In reality, Jackal has only two motors, one per side. However, it's more
+         straightforward for Gazebo to simulate as if there's an actuator per wheel. -->
+    <transmission name="${prefix}_wheel_trans">
+      <type>transmission_interface/SimpleTransmission</type>
+      <joint name="${prefix}_wheel">
+        <hardwareInterface>hardware_interface/VelocityJointInterface</hardwareInterface>
+      </joint>
+      <actuator name="${prefix}_actuator">
+        <mechanicalReduction>1</mechanicalReduction>
+      </actuator>
+    </transmission>
+  </xacro:macro>
   <xacro:wheel prefix="front_left">
     <origin xyz="${wheelbase/2} ${track/2} ${wheel_vertical_offset}" rpy="0 0 0" />
@@ -66,5 +112,5 @@
       <origin xyz="0 0 ${footprint_vertical_offset}" rpy="${pi/2} 0 ${pi/2}"/>
       <geometry>
-        <mesh filename="file://$(find nanovoxmap_example)/meshes/jackal-fenders.stl"/>
+        <mesh filename="package://nanovoxmap_example/meshes/jackal-fenders.stl"/>
       </geometry>
       <material name="yellow" />
@@ -75,4 +121,7 @@
     <child link="fenders_link" />
   </joint>
+  <gazebo reference="fenders_link">
+    <material>Gazebo/Yellow</material>
+  </gazebo>
   <link name="mid_mount"></link>
   <joint name="mid_mount_joint" type="fixed">
@@ -81,43 +130,25 @@
     <origin xyz="0 0 ${chassis_height}" />
   </joint>
-  <!-- Gazebo plugin for differential drive -->
+  <!-- Bring in simulation data for Gazebo. -->
   <gazebo>
-    <plugin filename="gz-sim-diff-drive-system" name="gz::sim::systems::DiffDrive">
-      <odom_publisher_frequency>500</odom_publisher_frequency>
-      <left_joint>rear_left_wheel_joint</left_joint>
-      <left_joint>front_left_wheel_joint</left_joint>
-      <right_joint>rear_right_wheel_joint</right_joint>
-      <right_joint>front_right_wheel_joint</right_joint>
-      <wheel_radius>0.098</wheel_radius>
-      <wheel_separation>0.37559</wheel_separation>
-      <max_linear_velocity>10.0</max_linear_velocity>
-      <max_angular_velocity>10.0</max_angular_velocity>
-      <topic>/jackal/cmd_vel</topic>
-      <child_frame_id>base_link</child_frame_id>
+    <plugin name="gazebo_ros_control" filename="libgazebo_ros_control.so">
+      <robotNamespace>/</robotNamespace>
     </plugin>
   </gazebo>
-  <!-- Ground truth -->
+  <!-- Ground Truth -->
   <gazebo>
-    <plugin filename="gz-sim-odometry-publisher-system" name="gz::sim::systems::OdometryPublisher">
-      <odom_topic>jackal/ground_truth</odom_topic>
-      <odom_frame>world</odom_frame>
-      <robot_base_frame>base_link</robot_base_frame>
-      <odom_publish_frequency>500</odom_publish_frequency>
-      <dimensions>3</dimensions>
-    </plugin>
-  </gazebo>
-  <!-- Joint States publisher -->
-  <gazebo>
-    <plugin filename="gz-sim-joint-state-publisher-system" name="gz::sim::systems::JointStatePublisher">
-      <topic>joint_states</topic>
-      <joint_name>front_left_wheel_joint</joint_name>
-      <joint_name>rear_left_wheel_joint</joint_name>
-      <joint_name>front_right_wheel_joint</joint_name>
-      <joint_name>rear_right_wheel_joint</joint_name>
+    <plugin name="jackal_odometry" filename="libgazebo_ros_p3d.so">
+      <alwaysOn>true</alwaysOn>
+      <updateRate>100.0</updateRate>
+      <frameName>world</frameName>
+      <bodyName>base_link</bodyName>
+      <topicName>jackal/ground_truth</topicName>
+      <gaussianNoise>0.00</gaussianNoise>
+      <xyzOffsets>0 0 0</xyzOffsets>
+      <rpyOffsets>0 0 0</rpyOffsets>
     </plugin>
   </gazebo>
   <!-- Lidar -->
-  <xacro:include filename="$(find nanovoxmap_example)/urdf/lidar.xacro" />
-  <!-- Depth Camera -->
-  <xacro:include filename="$(find nanovoxmap_example)/urdf/depth_camera.xacro" />
+  <xacro:include filename="$(find nanovoxmap_example)/urdf/Lidar.xacro"/>
+  <xacro:include filename="$(find nanovoxmap_example)/urdf/depth_camera.xacro"/>
 </robot>
